File: GPIO_UNIT/CPU.kicad_sch (KiCad schematic)
At the start: 8 parts, among them SW202 default_switch, U201 HEADER_3x2, U202 ATmega328-A, Y201 Crystal_GND2

Commit message: Digital pins are now able to use the analog pinnumbering as well. Pin can be set to an analog or digital pin number by simply pressing a or d respectively when editting the pinnumbers. Take note that one can fill in invalid analog pinnumbers. Also due to me support the arduino mega, I should remove pin number limit all togather.
Parts:
- removed SW202: default_switch, custom_kicad_lib_sk:default_switch, symbol custom_kicad_lib_sk:default_switch
- added SW202: SW_Push, custom_kicad_lib_sk:tactile_SMD_6mm, symbol custom_kicad_lib_sk:tactile_SMD_6mm
Connections:
- net GND: now also SW202.1
- net RESET: now also SW202.2
Changed lines of the file:
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@@
     )
   )
-  (symbol (lib_id "custom_kicad_lib_sk:default_switch") (at 111.76 129.54 90) (unit 1)
-    (in_bom yes) (on_board yes) (dnp no)
+  (symbol (lib_id "custom_kicad_lib_sk:tactile_SMD_6mm") (at 111.76 129.54 90) (unit 1)
+    (in_bom yes) (on_board yes) (dnp no) (fields_autoplaced)
     (property "Reference" "SW202" (at 113.03 128.27 90)
       (effects (font (size 1.27 1.27)) (justify right))
     )
-    (property "Value" "default_switch" (at 113.03 130.81 90)
+    (property "Value" "SW_Push" (at 113.03 130.81 90)
       (effects (font (size 1.27 1.27)) (justify right))
     )
-    (property "Footprint" "custom_kicad_lib_sk:default_switch" (at 119.38 129.54 0)
+    (property "Footprint" "custom_kicad_lib_sk:tactile_SMD_6mm" (at 106.68 129.54 0)
       (effects (font (size 1.27 1.27)) hide)
     )
-    (property "Datasheet" "~" (at 111.76 129.54 0)
+    (property "Datasheet" "~" (at 106.68 129.54 0)
       (effects (font (size 1.27 1.27)) hide)
     )
-    (property "JLCPCB Part#" "C318884" (at 113.03 132.08 90)
-      (effects (font (size 1.27 1.27)) (justify right) hide)
+    (property "JLCPCB Part#" "C294567" (at 111.76 129.54 0)
+      (effects (font (size 1.27 1.27)) hide)
     )
+    (pin "2")
     (pin "1")
-    (pin "2")
     (instances
       (project "GPIO_UNIT"
@@
           (reference "SW202") (unit 1)
         )
-      )
-      (project "atmega328"
-        (path "/8e079fd1-98e3-4beb-9638-08f2e3990e09"
-          (reference "SW202") (unit 1)
-        )
