File: GPIO_UNIT/switches.kicad_sch (KiCad schematic)
At the start: 5 parts, among them J801 Screw_Terminal_01x05, SW801 SW_Push, SW802 SW_Push, SW803 SW_Push, SW804 SW_Push

Commit message: Digital pins are now able to use the analog pinnumbering as well. Pin can be set to an analog or digital pin number by simply pressing a or d respectively when editting the pinnumbers. Take note that one can fill in invalid analog pinnumbers. Also due to me support the arduino mega, I should remove pin number limit all togather.
Parts:
- removed J801: Screw_Terminal_01x05, TerminalBlock_Phoenix:TerminalBlock_Phoenix_MKDS-1,5-5-5.08_1x05_P5.08mm_Horizontal, symbol Connector:Screw_Terminal_01x05
- added J802, J803, J804, J805: Conn_01x03_Pin, Connector_PinHeader_2.54mm:PinHeader_1x03_P2.54mm_Vertical, symbol Connector:Conn_01x03_Pin
- added J806: Conn_01x01_Pin, Connector_PinHeader_2.54mm:PinHeader_1x01_P2.54mm_Vertical, symbol Connector:Conn_01x01_Pin
Connections:
- net GND: now also J802.1 (Pin_1), J803.1 (Pin_1), J804.1 (Pin_1), J805.1 (Pin_1), J806.1 (Pin_1)
- net SW1: now also J802.3 (Pin_3)
- net SW2: now also J803.3 (Pin_3)
- net SW3: now also J804.3 (Pin_3)
- net SW4: now also J805.3 (Pin_3)
- new net +5V: J802.2 (Pin_2), J803.2 (Pin_2), J804.2 (Pin_2), J805.2 (Pin_2)
Other:
- note added: "extra gnd pin for CS add-on board"
