File: HARDWARE/GPIO_UNIT/CPU.kicad_sch (KiCad schematic)
At the start: 8 parts, among them SW202 SW_Push, U201 HEADER_3x2, U202 ATmega328-A, Y201 Crystal_GND2

Commit message: added GPIO UNIT board. To be renamed Jack Of All trades
Connections:
- net reset is gone; now on net RESET: U202.29 (~{RESET}/PC6)
Changed lines of the file:
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@@
-    (effects (font (size 1.27 1.27)) (justify left bottom))
-  )
-  (label "reset" (at 186.69 91.44 0) (fields_autoplaced)
     (effects (font (size 1.27 1.27)) (justify left bottom))
   )
@@
     (effects (font (size 1.27 1.27)) (justify right))
   )
+  (hierarchical_label "RESET" (shape input) (at 186.69 91.44 0) (fields_autoplaced)
+    (effects (font (size 1.27 1.27)) (justify left))
+  )
   (hierarchical_label "D6" (shape bidirectional) (at 186.69 111.76 0) (fields_autoplaced)
