File: HARDWARE/GPIO_UNIT/LED.kicad_sch (KiCad schematic)
At the start: 16 parts, among them J901 Screw_Terminal_01x04, Q901 AO3400A, Q902 AO3400A, Q903 AO3400A

Commit message: added GPIO UNIT board. To be renamed Jack Of All trades
Parts:
- added D904, D905, D906: 1N4148WS, Diode_SMD:D_SOD-323, symbol custom_kicad_lib_sk:1N4148WS
- J901: value Screw_Terminal_01x04 -> Screw_Terminal_01x05; footprint TerminalBlock_Phoenix:TerminalBlock_Phoenix_MPT-0,5-4-2.54_1x04_P2.54mm_Horizontal -> TerminalBlock_Phoenix:TerminalBlock_Phoenix_MPT-0,5-5-2.54_1x05_P2.54mm_Horizontal; symbol Connector:Screw_Terminal_01x04 -> Connector:Screw_Terminal_01x05
Connections:
- net GND: now also J901.1 (Pin_1)
- net VCC: now also J901.5 (Pin_5), D904.1 (K), D905.1 (K), D906.1 (K); no longer J901.4 (Pin_4)
- net at Q903.3 (D): now also J901.2 (Pin_2), D906.2 (A); no longer J901.1 (Pin_1)
- net at Q902.3 (D): now also J901.3 (Pin_3), D905.2 (A); no longer J901.2 (Pin_2)
- net at Q901.3 (D): now also J901.4 (Pin_4), D904.2 (A); no longer J901.3 (Pin_3)
