File: HARDWARE/GPIO_UNIT/USB.kicad_sch (KiCad schematic)
At the start: 14 parts, among them J701 USB_B_Mini, U701 CH340G, Y701 Crystal

Commit message: added GPIO UNIT board. To be renamed Jack Of All trades
Parts:
- J301: renamed from J?; footprint (none) -> Connector_PinHeader_2.54mm:PinHeader_1x03_P2.54mm_Horizontal
- gave numbers to parts that had none: 2
Changed lines of the file:
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@@
   (symbol (lib_id "resistors_0603:R_100R_0603") (at 144.78 62.23 90) (unit 1)
     (in_bom yes) (on_board yes) (dnp no)
-    (property "Reference" "R?" (at 140.97 63.5 90)
+    (property "Reference" "R301" (at 140.97 63.5 90)
       (effects (font (size 1.27 1.27)))
     )
@@
       (project "GPIO_UNIT"
         (path "/4337ba29-1ab5-4e01-8f76-ba2df9f917ea/a906ae47-0b9b-4d87-b0df-13938bf2addd"
-          (reference "R?") (unit 1)
+          (reference "R301") (unit 1)
         )
       )
@@
   (symbol (lib_id "resistors_0603:R_100R_0603") (at 144.78 64.77 90) (unit 1)
     (in_bom yes) (on_board yes) (dnp no)
-    (property "Reference" "R?" (at 140.97 66.04 90)
+    (property "Reference" "R302" (at 140.97 66.04 90)
       (effects (font (size 1.27 1.27)))
     )
@@
       (project "GPIO_UNIT"
         (path "/4337ba29-1ab5-4e01-8f76-ba2df9f917ea/a906ae47-0b9b-4d87-b0df-13938bf2addd"
-          (reference "R?") (unit 1)
+          (reference "R302") (unit 1)
         )
       )
@@
   (symbol (lib_id "Connector:Conn_01x03_Pin") (at 134.62 64.77 0) (mirror x) (unit 1)
     (in_bom yes) (on_board yes) (dnp no)
-    (property "Reference" "J?" (at 135.89 68.58 0)
+    (property "Reference" "J301" (at 135.89 68.58 0)
       (effects (font (size 1.27 1.27)))
     )
@@
       (effects (font (size 1.27 1.27)) hide)
     )
-    (property "Footprint" "" (at 134.62 64.77 0)
+    (property "Footprint" "Connector_PinHeader_2.54mm:PinHeader_1x03_P2.54mm_Horizontal" (at 134.62 64.77 0)
       (effects (font (size 1.27 1.27)) hide)
     )
@@
       (project "GPIO_UNIT"
         (path "/4337ba29-1ab5-4e01-8f76-ba2df9f917ea/a906ae47-0b9b-4d87-b0df-13938bf2addd"
-          (reference "J?") (unit 1)
-        )
-      )
+          (reference "J301") (unit 1)
+        )
+      )
